File: serial.brd (EAGLE design)
At the start: 70.8 x 25.4 mm, 12 parts, among them IC1 74AC164D, IC2 74AC164D, IC3 74AC164D

Commit message: Test update. Not worth mentioning.
Connections:
- net GND renamed UPS
Routing:
- net UPS: track 76.3 -> 67.2 mm, vias 38 -> 0
- removed copper zone on layer 1, net UPS
- removed copper zone on layer 16, net UPS
Changed lines of the file:
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@@
 <?xml version="1.0" encoding="utf-8"?>
 <!DOCTYPE eagle SYSTEM "eagle.dtd">
-<eagle version="6.2">
+<eagle version="6.4">
 <drawing>
 <settings>
@@
 </class>
 </classes>
-<designrules>
+<designrules name="default">
 <description language="en">&lt;b&gt;EAGLE Design Rules&lt;/b&gt;
 &lt;p&gt;
@@
 </elements>
 <signals>
-<signal name="GND">
+<signal name="UPS">
 <contactref element="IC1" pad="7"/>
 <contactref element="IC2" pad="7"/>
@@
 <wire x1="17.78" y1="15.24" x2="19.05" y2="13.97" width="0.3048" layer="1"/>
 <wire x1="17.78" y1="15.24" x2="17.2466" y2="15.24" width="0.3048" layer="1"/>
-<wire x1="15.24" y1="21.59" x2="17.2466" y2="21.59" width="0.3048" layer="1"/>
-<wire x1="10.16" y1="16.51" x2="15.24" y2="21.59" width="0.3048" layer="1"/>
 <wire x1="33.02" y1="21.59" x2="33.7566" y2="21.59" width="0.3048" layer="1"/>
 <wire x1="30.48" y1="19.05" x2="33.02" y2="21.59" width="0.3048" layer="1"/>
@@
 <wire x1="52.07" y1="21.59" x2="52.8066" y2="21.59" width="0.3048" layer="1"/>
 <wire x1="45.72" y1="15.24" x2="52.07" y2="21.59" width="0.3048" layer="1"/>
-<polygon width="0.4064" layer="16">
-<vertex x="6.35" y="34.29"/>
-<vertex x="76.2" y="34.29"/>
-<vertex x="76.2" y="10.16"/>
-<vertex x="6.35" y="10.16"/>
-</polygon>
-<polygon width="0.4064" layer="1">
-<vertex x="6.35" y="34.29"/>
-<vertex x="76.2" y="34.29"/>
-<vertex x="76.2" y="10.16"/>
-<vertex x="6.35" y="10.16"/>
-</polygon>
-<via x="11.43" y="26.67" extent="1-16" drill="0.6" shape="square"/>
-<via x="10.16" y="30.48" extent="1-16" drill="0.6" shape="square"/>
-<via x="7.62" y="27.94" extent="1-16" drill="0.6" shape="square"/>
-<via x="7.62" y="33.02" extent="1-16" drill="0.6" shape="square"/>
-<via x="7.62" y="24.13" extent="1-16" drill="0.6" shape="square"/>
-<via x="7.62" y="12.7" extent="1-16" drill="0.6" shape="square"/>
-<via x="10.16" y="11.43" extent="1-16" drill="0.6" shape="square"/>
-<via x="13.97" y="11.43" extent="1-16" drill="0.6" shape="square"/>
-<via x="17.78" y="11.43" extent="1-16" drill="0.6" shape="square"/>
-<via x="21.59" y="11.43" extent="1-16" drill="0.6" shape="square"/>
-<via x="25.4" y="11.43" extent="1-16" drill="0.6" shape="square"/>
-<via x="29.21" y="11.43" extent="1-16" drill="0.6" shape="square"/>
-<via x="33.02" y="11.43" extent="1-16" drill="0.6" shape="square"/>
-<via x="36.83" y="11.43" extent="1-16" drill="0.6" shape="square"/>
-<via x="27.94" y="24.13" extent="1-16" drill="0.6" shape="square"/>
-<via x="44.45" y="25.4" extent="1-16" drill="0.6" shape="square"/>
-<via x="40.64" y="24.13" extent="1-16" drill="0.6" shape="square"/>
-<via x="33.02" y="26.67" extent="1-16" drill="0.6" shape="square"/>
-<via x="49.53" y="22.86" extent="1-16" drill="0.6" shape="square"/>
-<via x="66.04" y="25.4" extent="1-16" drill="0.6" shape="square"/>
-<via x="69.85" y="25.4" extent="1-16" drill="0.6" shape="square"/>
-<via x="73.66" y="25.4" extent="1-16" drill="0.6" shape="square"/>
-<via x="73.66" y="27.94" extent="1-16" drill="0.6" shape="square"/>
-<via x="73.66" y="30.48" extent="1-16" drill="0.6" shape="square"/>
-<via x="71.12" y="31.75" extent="1-16" drill="0.6" shape="square"/>
-<via x="67.31" y="31.75" extent="1-16" drill="0.6" shape="square"/>
-<via x="40.64" y="11.43" extent="1-16" drill="0.6" shape="square"/>
-<via x="44.45" y="11.43" extent="1-16" drill="0.6" shape="square"/>
-<via x="48.26" y="11.43" extent="1-16" drill="0.6" shape="square"/>
-<via x="52.07" y="11.43" extent="1-16" drill="0.6" shape="square"/>
-<via x="55.88" y="11.43" extent="1-16" drill="0.6" shape="square"/>
-<via x="59.69" y="11.43" extent="1-16" drill="0.6" shape="square"/>
-<via x="63.5" y="11.43" extent="1-16" drill="0.6" shape="square"/>
-<via x="67.31" y="11.43" extent="1-16" drill="0.6" shape="square"/>
-<via x="71.12" y="11.43" extent="1-16" drill="0.6" shape="square"/>
-<via x="74.93" y="11.43" extent="1-16" drill="0.6" shape="square"/>
-<via x="17.78" y="26.67" extent="1-16" drill="0.6" shape="square"/>
-<via x="20.32" y="27.94" extent="1-16" drill="0.6" shape="square"/>
+<wire x1="17.78" y1="15.24" x2="17.2466" y2="21.59" width="0" layer="19" extent="1-1"/>
 </signal>
 <signal name="VCC">
