File: serial.sch (EAGLE design)
At the start: 12 parts, among them IC1 74AC164D, IC2 74AC164D, IC3 74AC164D

Commit message: Test update. Not worth mentioning.
Connections:
- net GND renamed UPS
Changed lines of the file:
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@@
 <?xml version="1.0" encoding="utf-8"?>
 <!DOCTYPE eagle SYSTEM "eagle.dtd">
-<eagle version="6.2">
+<eagle version="6.4">
 <drawing>
 <settings>
@@
 </segment>
 </net>
-<net name="GND" class="0">
+<net name="UPS" class="0">
 <segment>
 <pinref part="IC1" gate="A" pin="B"/>
